File: Projects/_Dev Boards/Type-C Power port/board-Type-C-31-M-17.sch (EAGLE design)
At the start: 2 parts, among them J1 USB-TYPE-C-31-M-17

Commit message: update
Parts:
- added R1, R2: 5.1k, angrypig7-RCL:RR0603
- JP1: device pinhead_v2:PINHD-1X4/OCT -> angrypig7-Connectors-PinHeads:PINHD-1X4
Connections:
- removed net N$3: J1.CC1, JP1.2
- removed net N$4: J1.CC2, JP1.3
- new net GND: J1.GND, J1.SHIELD, JP1.3, JP1.4, R1.2, R2.2
- new net VBUS: J1.VBUS, JP1.1, JP1.2
- net N$1: now also J1.CC1, R1.1; no longer J1.GND, J1.SHIELD, JP1.4
- net N$2: now also J1.CC2, R2.1; no longer J1.VBUS, JP1.1
Other:
- moved on the sheet: JP1
Changed lines of the file:
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@@
 <?xml version="1.0" encoding="utf-8"?>
 <!DOCTYPE eagle SYSTEM "eagle.dtd">
-<eagle version="9.6.1">
+<eagle version="9.6.2">
 <drawing>
 <settings>
@@
 <setting verticaltext="up"/>
 </settings>
-<grid distance="0.1" unitdist="inch" unit="inch" style="lines" multiple="1" display="no" altdistance="0.01" altunitdist="inch" altunit="inch"/>
+<grid distance="50" unitdist="mil" unit="mil" style="lines" multiple="1" display="no" altdistance="0.01" altunitdist="inch" altunit="inch"/>
 <layers>
 <layer number="1" name="Top" color="4" fill="1" visible="no" active="no"/>
@@
 <class number="0" name="default" width="0.254" drill="0">
 </class>
-<class number="1" name="power" width="0.4572" drill="0">
+<class number="1" name="power" width="0.4064" drill="0">
 </class>
 </classes>
 <parts>
-<part name="J1" library="angrypig7-Connectors" deviceset="USB-TYPE-C-31-M-17" device=""/>
-<part name="JP1" library="pinhead_v2" deviceset="PINHD-1X4" device="/OCT"/>
+<part name="R1" library="angrypig7-RCL" deviceset="R" device="R0603" package3d_urn="urn:adsk.eagle:package:23555/54" value="5.1k"/>
+<part name="R2" library="angrypig7-RCL" deviceset="R" device="R0603" package3d_urn="urn:adsk.eagle:package:23555/54" value="5.1k"/>
+<part name="J1" library="angrypig7-Connectors" deviceset="USB-TYPE-C-31-M-17" device="" package3d_urn="urn:adsk.eagle:package:24334504/2"/>
+<part name="JP1" library="angrypig7-Connectors-PinHeads" deviceset="PINHD-1X4" device="" package3d_urn="urn:adsk.eagle:package:22407/2"/>
 </parts>
 <sheets>
@@
 </plain>
 <instances>
-<instance part="J1" gate="G$1" x="7.62" y="20.32" smashed="yes">
+<instance part="R1" gate="G$1" x="33.02" y="22.86" smashed="yes">
+<attribute name="NAME" x="27.178" y="23.0886" size="1.778" layer="95"/>
+<attribute name="VALUE" x="35.687" y="23.114" size="1.778" layer="96"/>
+</instance>
+<instance part="R2" gate="G$1" x="33.02" y="20.32" smashed="yes">
+<attribute name="NAME" x="27.178" y="20.5486" size="1.778" layer="95"/>
+<attribute name="VALUE" x="35.687" y="20.574" size="1.778" layer="96"/>
+</instance>
+<instance part="J1" gate="G$1" x="12.7" y="21.59" smashed="yes">
 <attribute name="NAME" x="6.35" y="28.194" size="1.27" layer="95"/>
 </instance>
-<instance part="JP1" gate="A" x="43.18" y="20.32" smashed="yes">
-<attribute name="NAME" x="36.83" y="28.575" size="1.778" layer="95"/>
-<attribute name="VALUE" x="36.83" y="12.7" size="1.778" layer="96"/>
+<instance part="JP1" gate="A" x="54.61" y="22.86" smashed="yes">
+<attribute name="NAME" x="48.26" y="31.115" size="1.778" layer="95"/>
+<attribute name="VALUE" x="48.26" y="17.78" size="1.778" layer="96"/>
 </instance>
 </instances>
@@
 </busses>
 <nets>
-<net name="N$1" class="1">
-<segment>
-<pinref part="J1" gate="G$1" pin="SHIELD"/>
+<net name="GND" class="1">
+<segment>
 <wire x1="7.62" y1="10.16" x2="7.62" y2="7.62" width="0.1524" layer="91"/>
 <wire x1="7.62" y1="7.62" x2="30.48" y2="7.62" width="0.1524" layer="91"/>
 <wire x1="30.48" y1="7.62" x2="30.48" y2="17.78" width="0.1524" layer="91"/>
-<pinref part="J1" gate="G$1" pin="GND"/>
 <wire x1="30.48" y1="17.78" x2="25.4" y2="17.78" width="0.1524" layer="91"/>
-<pinref part="JP1" gate="A" pin="4"/>
 <wire x1="30.48" y1="17.78" x2="40.64" y2="17.78" width="0.1524" layer="91"/>
 <junction x="30.48" y="17.78"/>
-</segment>
-</net>
-<net name="N$2" class="1">
-<segment>
+<pinref part="J1" gate="G$1" pin="GND"/>
+<pinref part="J1" gate="G$1" pin="SHIELD"/>
+<pinref part="R2" gate="G$1" pin="2"/>
+<wire x1="38.1" y1="20.32" x2="40.64" y2="20.32" width="0.1524" layer="91"/>
+<wire x1="40.64" y1="20.32" x2="40.64" y2="17.78" width="0.1524" layer="91"/>
+<pinref part="R1" gate="G$1" pin="2"/>
+<wire x1="38.1" y1="22.86" x2="40.64" y2="22.86" width="0.1524" layer="91"/>
+<wire x1="40.64" y1="22.86" x2="40.64" y2="20.32" width="0.1524" layer="91"/>
+<junction x="40.64" y="20.32"/>
+<pinref part="JP1" gate="A" pin="3"/>
+<wire x1="40.64" y1="22.86" x2="46.99" y2="22.86" width="0.1524" layer="91"/>
+<junction x="40.64" y="22.86"/>
+<pinref part="JP1" gate="A" pin="4"/>
+<wire x1="46.99" y1="22.86" x2="52.07" y2="22.86" width="0.1524" layer="91"/>
+<wire x1="46.99" y1="22.86" x2="46.99" y2="20.32" width="0.1524" layer="91"/>
+<wire x1="46.99" y1="20.32" x2="52.07" y2="20.32" width="0.1524" layer="91"/>
+<junction x="46.99" y="22.86"/>
+</segment>
+</net>
+<net name="VBUS" class="1">
+<segment>
+<wire x1="25.4" y1="25.4" x2="46.99" y2="25.4" width="0.1524" layer="91"/>
 <pinref part="J1" gate="G$1" pin="VBUS"/>
+<pinref part="JP1" gate="A" pin="2"/>
 <pinref part="JP1" gate="A" pin="1"/>
-<wire x1="25.4" y1="25.4" x2="40.64" y2="25.4" width="0.1524" layer="91"/>
-</segment>
-</net>
-<net name="N$3" class="0">
-<segment>
+<wire x1="46.99" y1="25.4" x2="52.07" y2="25.4" width="0.1524" layer="91"/>
+<wire x1="52.07" y1="27.94" x2="46.99" y2="27.94" width="0.1524" layer="91"/>
+<wire x1="46.99" y1="27.94" x2="46.99" y2="25.4" width="0.1524" layer="91"/>
+<junction x="46.99" y="25.4"/>
+</segment>
+</net>
+<net name="N$1" class="0">
+<segment>
+<pinref part="R1" gate="G$1" pin="1"/>
 <pinref part="J1" gate="G$1" pin="CC1"/>
-<pinref part="JP1" gate="A" pin="2"/>
-<wire x1="25.4" y1="22.86" x2="40.64" y2="22.86" width="0.1524" layer="91"/>
-</segment>
-</net>
-<net name="N$4" class="0">
+<wire x1="27.94" y1="22.86" x2="25.4" y2="22.86" width="0.1524" layer="91"/>
+</segment>
+</net>
+<net name="N$2" class="0">
 <segment>
 <pinref part="J1" gate="G$1" pin="CC2"/>
-<pinref part="JP1" gate="A" pin="3"/>
-<wire x1="25.4" y1="20.32" x2="40.64" y2="20.32" width="0.1524" layer="91"/>
+<pinref part="R2" gate="G$1" pin="1"/>
+<wire x1="25.4" y1="20.32" x2="27.94" y2="20.32" width="0.1524" layer="91"/>
 </segment>
 </net>
@@
 </schematic>
 </drawing>
+<compatibility>
+<note version="8.3" severity="warning">
+Since Version 8.3, EAGLE supports URNs for individual library
+assets (packages, symbols, and devices). The URNs of those assets
+will not be understood (or retained) with this version.
+</note>
+<note version="8.3" severity="warning">
+Since Version 8.3, EAGLE supports the association of 3D packages
+with devices in libraries, schematics, and board files. Those 3D
+packages will not be understood (or retained) with this version.
+</note>
+<note version="8.4" severity="warning">
+Since Version 8.4, EAGLE supports properties for SPICE simulation.
+Probes in schematics and SPICE mapping objects found in parts and library devices
+will not be understood with this version. Update EAGLE to the latest version
+for full support of SPICE simulation.
+</note>
+</compatibility>
 </eagle>
